File: schema.sch (EAGLE design)
At the start: 7 parts, among them X1 BU-SMA-G

Commit message: Pin swap issue on FX758 fixed
Parts:
- TRANSMITTER: device hi-link:FX758 -> custom-parts:FX758
Other:
- moved on the sheet: TRANSMITTER
Changed lines of the file:
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@@
 <?xml version="1.0" encoding="utf-8"?>
 <!DOCTYPE eagle SYSTEM "eagle.dtd">
-<eagle version="8.1.1">
+<eagle version="8.2.1">
 <drawing>
 <settings>
@@
 </classes>
 <parts>
-<part name="TRANSMITTER" library="hi-link" deviceset="FX758" device=""/>
 <part name="X1" library="con-coax" deviceset="BU-SMA-G" device=""/>
 <part name="GND1" library="supply1" deviceset="GND" device=""/>
@@
 <part name="P+2" library="supply1" deviceset="+5V" device=""/>
 <part name="GND4" library="supply1" deviceset="GND" device=""/>
+<part name="TRANSMITTER" library="custom-parts" deviceset="FX758" device=""/>
 </parts>
 <sheets>
@@
 </plain>
 <instances>
-<instance part="TRANSMITTER" gate="G$1" x="0" y="0"/>
 <instance part="X1" gate="G1" x="-43.18" y="5.08"/>
 <instance part="GND1" gate="1" x="-38.1" y="0"/>
@@
 <instance part="P+2" gate="1" x="7.62" y="-27.94" rot="R180"/>
 <instance part="GND4" gate="1" x="5.08" y="-30.48"/>
+<instance part="TRANSMITTER" gate="G$1" x="0" y="0"/>
 </instances>
 <busses>
@@
 <wire x1="-17.78" y1="7.62" x2="-25.4" y2="7.62" width="0.1524" layer="91"/>
 <wire x1="-25.4" y1="7.62" x2="-25.4" y2="2.54" width="0.1524" layer="91"/>
-<pinref part="TRANSMITTER" gate="G$1" pin="GND@2"/>
 <wire x1="-25.4" y1="2.54" x2="-17.78" y2="2.54" width="0.1524" layer="91"/>
 <pinref part="GND3" gate="1" pin="GND"/>
 <junction x="-25.4" y="2.54"/>
 <pinref part="TRANSMITTER" gate="G$1" pin="GND@1"/>
+<pinref part="TRANSMITTER" gate="G$1" pin="GND@2"/>
 </segment>
 <segment>
@@
 </segment>
 <segment>
-<pinref part="TRANSMITTER" gate="G$1" pin="GND@3"/>
 <wire x1="17.78" y1="0" x2="20.32" y2="0" width="0.1524" layer="91"/>
 <wire x1="20.32" y1="0" x2="20.32" y2="-5.08" width="0.1524" layer="91"/>
-<pinref part="TRANSMITTER" gate="G$1" pin="GND@4"/>
 <wire x1="20.32" y1="-5.08" x2="17.78" y2="-5.08" width="0.1524" layer="91"/>
 <pinref part="GND5" gate="1" pin="GND"/>
@@
 <pinref part="CAM-SUPPLY" gate="G$1" pin="2"/>
 <wire x1="20.32" y1="-5.08" x2="45.72" y2="-5.08" width="0.1524" layer="91"/>
+<pinref part="TRANSMITTER" gate="G$1" pin="GND@3"/>
+<pinref part="TRANSMITTER" gate="G$1" pin="GND@4"/>
 </segment>
 <segment>
@@
 <segment>
 <pinref part="X1" gate="G1" pin="1"/>
+<wire x1="-40.64" y1="5.08" x2="-17.78" y2="5.08" width="0.1524" layer="91"/>
 <pinref part="TRANSMITTER" gate="G$1" pin="ANT"/>
-<wire x1="-40.64" y1="5.08" x2="-17.78" y2="5.08" width="0.1524" layer="91"/>
 </segment>
 </net>
@@
 <segment>
 <pinref part="CH-SEL" gate="1" pin="4"/>
+<wire x1="-17.78" y1="-10.16" x2="-17.78" y2="-5.08" width="0.1524" layer="91"/>
 <pinref part="TRANSMITTER" gate="G$1" pin="CS1"/>
-<wire x1="-17.78" y1="-10.16" x2="-17.78" y2="-5.08" width="0.1524" layer="91"/>
 </segment>
 </net>
 <net name="CH2" class="0">
 <segment>
-<pinref part="TRANSMITTER" gate="G$1" pin="CS2"/>
 <pinref part="CH-SEL" gate="1" pin="5"/>
 <wire x1="-17.78" y1="-2.54" x2="-20.32" y2="-2.54" width="0.1524" layer="91"/>
 <wire x1="-20.32" y1="-2.54" x2="-20.32" y2="-10.16" width="0.1524" layer="91"/>
+<pinref part="TRANSMITTER" gate="G$1" pin="CS2"/>
 </segment>
 </net>
 <net name="CH3" class="0">
 <segment>
-<pinref part="TRANSMITTER" gate="G$1" pin="CS3"/>
 <pinref part="CH-SEL" gate="1" pin="6"/>
 <wire x1="-17.78" y1="0" x2="-22.86" y2="0" width="0.1524" layer="91"/>
 <wire x1="-22.86" y1="0" x2="-22.86" y2="-10.16" width="0.1524" layer="91"/>
+<pinref part="TRANSMITTER" gate="G$1" pin="CS3"/>
 </segment>
 </net>
 <net name="VIDEO-IN" class="0">
 <segment>
-<pinref part="TRANSMITTER" gate="G$1" pin="VIN"/>
 <pinref part="VIDEO-IN" gate="G$1" pin="1"/>
 <wire x1="17.78" y1="5.08" x2="22.86" y2="5.08" width="0.1524" layer="91"/>
 <wire x1="22.86" y1="5.08" x2="22.86" y2="15.24" width="0.1524" layer="91"/>
+<pinref part="TRANSMITTER" gate="G$1" pin="VIN"/>
 </segment>
 </net>
 <net name="AUDIO-IN" class="0">
 <segment>
-<pinref part="TRANSMITTER" gate="G$1" pin="A6.5"/>
 <pinref part="AUDIO-IN" gate="G$1" pin="1"/>
 <wire x1="17.78" y1="2.54" x2="30.48" y2="2.54" width="0.1524" layer="91"/>
+<pinref part="TRANSMITTER" gate="G$1" pin="A6.5"/>
 </segment>
 </net>
 <net name="+5V" class="0">
 <segment>
-<pinref part="TRANSMITTER" gate="G$1" pin="+5V"/>
 <pinref part="CAM-SUPPLY" gate="G$1" pin="1"/>
 <wire x1="17.78" y1="-2.54" x2="33.02" y2="-2.54" width="0.1524" layer="91"/>
@@
 <wire x1="33.02" y1="-12.7" x2="33.02" y2="-2.54" width="0.1524" layer="91"/>
 <junction x="33.02" y="-2.54"/>
-</segment>
-<segment>
+<pinref part="TRANSMITTER" gate="G$1" pin="+5V"/>
+</segment>
+<segment>

Commit message: Minor adjustments
Parts:
- AUDIO-IN: value (none) -> A
- CAM-SUPPLY, PWR: value (none) -> G 5V
- VIDEO-IN: value (none) -> V
- renumbered X1 to SMA
Connections:
- net CH1: now also CH-SEL.1; no longer CH-SEL.4
- net CH2: now also CH-SEL.2; no longer CH-SEL.5
- net CH3: now also CH-SEL.3; no longer CH-SEL.6
- net GND: now also CH-SEL.4, CH-SEL.5, CH-SEL.6; no longer CH-SEL.1, CH-SEL.2, CH-SEL.3
Other:
- moved on the sheet: CH-SEL
Changed lines of the file:
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@@
 </classes>
 <parts>
-<part name="X1" library="con-coax" deviceset="BU-SMA-G" device=""/>
+<part name="SMA" library="con-coax" deviceset="BU-SMA-G" device=""/>
 <part name="GND1" library="supply1" deviceset="GND" device=""/>
 <part name="GND3" library="supply1" deviceset="GND" device=""/>
@@
 <part name="CH-SEL" library="switch-dil" deviceset="DP03" device=""/>
 <part name="GND2" library="supply1" deviceset="GND" device=""/>
-<part name="VIDEO-IN" library="pinhead" deviceset="PINHD-1X1" device=""/>
-<part name="AUDIO-IN" library="pinhead" deviceset="PINHD-1X1" device=""/>
-<part name="CAM-SUPPLY" library="pinhead" deviceset="PINHD-1X2" device=""/>
+<part name="VIDEO-IN" library="pinhead" deviceset="PINHD-1X1" device="" value="V"/>
+<part name="AUDIO-IN" library="pinhead" deviceset="PINHD-1X1" device="" value="A"/>
+<part name="CAM-SUPPLY" library="pinhead" deviceset="PINHD-1X2" device="" value="G  5V"/>
 <part name="P+1" library="supply1" deviceset="+5V" device=""/>
-<part name="PWR" library="pinhead" deviceset="PINHD-1X2" device=""/>
+<part name="PWR" library="pinhead" deviceset="PINHD-1X2" device="" value="G 5V"/>
 <part name="P+2" library="supply1" deviceset="+5V" device=""/>
 <part name="GND4" library="supply1" deviceset="GND" device=""/>
@@
 </plain>
 <instances>
-<instance part="X1" gate="G1" x="-43.18" y="5.08"/>
+<instance part="SMA" gate="G1" x="-43.18" y="5.08"/>
 <instance part="GND1" gate="1" x="-38.1" y="0"/>
 <instance part="GND3" gate="1" x="-25.4" y="0"/>
 <instance part="GND5" gate="1" x="20.32" y="-7.62"/>
-<instance part="CH-SEL" gate="1" x="-20.32" y="-17.78"/>
+<instance part="CH-SEL" gate="1" x="-20.32" y="-17.78" rot="R180"/>
 <instance part="GND2" gate="1" x="-22.86" y="-30.48"/>
 <instance part="VIDEO-IN" gate="G$1" x="22.86" y="17.78" rot="R90"/>
@@
 <segment>
 <pinref part="GND1" gate="1" pin="GND"/>
-<pinref part="X1" gate="G1" pin="2"/>
+<pinref part="SMA" gate="G1" pin="2"/>
 <wire x1="-38.1" y1="2.54" x2="-40.64" y2="2.54" width="0.1524" layer="91"/>
-</segment>
-<segment>
-<pinref part="GND2" gate="1" pin="GND"/>
-<pinref part="CH-SEL" gate="1" pin="1"/>
-<wire x1="-22.86" y1="-27.94" x2="-22.86" y2="-25.4" width="0.1524" layer="91"/>
-<pinref part="CH-SEL" gate="1" pin="3"/>
-<pinref part="CH-SEL" gate="1" pin="2"/>
-<wire x1="-17.78" y1="-25.4" x2="-20.32" y2="-25.4" width="0.1524" layer="91"/>
-<wire x1="-20.32" y1="-25.4" x2="-22.86" y2="-25.4" width="0.1524" layer="91"/>
-<junction x="-22.86" y="-25.4"/>
-<junction x="-20.32" y="-25.4"/>
 </segment>
 <segment>
@@
 <wire x1="5.08" y1="-27.94" x2="5.08" y2="-17.78" width="0.1524" layer="91"/>
 </segment>
+<segment>
+<pinref part="GND2" gate="1" pin="GND"/>
+<pinref part="CH-SEL" gate="1" pin="4"/>
+<wire x1="-22.86" y1="-27.94" x2="-22.86" y2="-25.4" width="0.1524" layer="91"/>
+<pinref part="CH-SEL" gate="1" pin="5"/>
+<wire x1="-22.86" y1="-25.4" x2="-20.32" y2="-25.4" width="0.1524" layer="91"/>
+<junction x="-22.86" y="-25.4"/>
+<pinref part="CH-SEL" gate="1" pin="6"/>
+<wire x1="-20.32" y1="-25.4" x2="-17.78" y2="-25.4" width="0.1524" layer="91"/>
+<junction x="-20.32" y="-25.4"/>
+</segment>
 </net>
 <net name="ANTENA" class="0">
 <segment>
-<pinref part="X1" gate="G1" pin="1"/>
+<pinref part="SMA" gate="G1" pin="1"/>
 <wire x1="-40.64" y1="5.08" x2="-17.78" y2="5.08" width="0.1524" layer="91"/>
 <pinref part="TRANSMITTER" gate="G$1" pin="ANT"/>
-</segment>
-</net>
-<net name="CH1" class="0">
-<segment>
-<pinref part="CH-SEL" gate="1" pin="4"/>
-<wire x1="-17.78" y1="-10.16" x2="-17.78" y2="-5.08" width="0.1524" layer="91"/>
-<pinref part="TRANSMITTER" gate="G$1" pin="CS1"/>
-</segment>
-</net>
-<net name="CH2" class="0">
-<segment>
-<pinref part="CH-SEL" gate="1" pin="5"/>
-<wire x1="-17.78" y1="-2.54" x2="-20.32" y2="-2.54" width="0.1524" layer="91"/>
-<wire x1="-20.32" y1="-2.54" x2="-20.32" y2="-10.16" width="0.1524" layer="91"/>
-<pinref part="TRANSMITTER" gate="G$1" pin="CS2"/>
-</segment>
-</net>
-<net name="CH3" class="0">
-<segment>
-<pinref part="CH-SEL" gate="1" pin="6"/>
-<wire x1="-17.78" y1="0" x2="-22.86" y2="0" width="0.1524" layer="91"/>
-<wire x1="-22.86" y1="0" x2="-22.86" y2="-10.16" width="0.1524" layer="91"/>
-<pinref part="TRANSMITTER" gate="G$1" pin="CS3"/>
 </segment>
 </net>
@@
 </segment>
 </net>
+<net name="CH1" class="0">
+<segment>
+<pinref part="TRANSMITTER" gate="G$1" pin="CS1"/>
+<pinref part="CH-SEL" gate="1" pin="1"/>
+<wire x1="-17.78" y1="-5.08" x2="-17.78" y2="-10.16" width="0.1524" layer="91"/>
+</segment>
+</net>
+<net name="CH2" class="0">
+<segment>
+<pinref part="TRANSMITTER" gate="G$1" pin="CS2"/>
+<pinref part="CH-SEL" gate="1" pin="2"/>
+<wire x1="-17.78" y1="-2.54" x2="-20.32" y2="-2.54" width="0.1524" layer="91"/>
+<wire x1="-20.32" y1="-2.54" x2="-20.32" y2="-10.16" width="0.1524" layer="91"/>
+</segment>
+</net>
+<net name="CH3" class="0">
+<segment>
+<pinref part="TRANSMITTER" gate="G$1" pin="CS3"/>
+<wire x1="-17.78" y1="0" x2="-22.86" y2="0" width="0.1524" layer="91"/>
+<wire x1="-22.86" y1="0" x2="-22.86" y2="-10.16" width="0.1524" layer="91"/>
+<pinref part="CH-SEL" gate="1" pin="3"/>
+</segment>
+</net>
